Commit message: ros2 control is modular, takes mock_components, real and isaac for control the so101

File: config/so101_new_calib.ros2_control.xacro (robot description, xacro)
@@ -1,18 +1,21 @@
 <?xml version="1.0"?>
 <robot xmlns:xacro="http://www.ros.org/wiki/xacro">
-    <xacro:macro name="so101_new_calib_ros2_control" params="name initial_positions_file">
+    <xacro:macro name="so101_new_calib_ros2_control" params="name initial_positions_file ros2_control_hardware_type">
         <xacro:property name="initial_positions" value="${xacro.load_yaml(initial_positions_file)['initial_positions']}"/>
         <ros2_control name="${name}" type="system">
             <hardware>
-                <!-- By default, set up controllers for simulation. This won't work on real hardware -->
-                <!-- <plugin>mock_components/GenericSystem</plugin> -->
-                <!-- Isaacsim -->
-                <!-- <plugin>topic_based_ros2_control/TopicBasedSystem</plugin>
-                <param name="joint_commands_topic">/isaac_joint_commands</param>
-                <param name="joint_states_topic">/isaac_joint_states</param> -->
-                <!-- Real Robot via Python Topic Interface -->
-                <plugin>topic_based_ros2_control/TopicBasedSystem</plugin>
-                <param name="joint_commands_topic">/real_joint_commands</param>
-                <param name="joint_states_topic">/real_joint_states</param>
+                <xacro:if value="${ros2_control_hardware_type == 'mock_components'}">
+                    <plugin>mock_components/GenericSystem</plugin>
+                </xacro:if>
+                <xacro:if value="${ros2_control_hardware_type == 'isaac'}">
+                    <plugin>topic_based_ros2_control/TopicBasedSystem</plugin>
+                    <param name="joint_commands_topic">/isaac_joint_commands</param>
+                    <param name="joint_states_topic">/isaac_joint_states</param>
+                </xacro:if>
+                <xacro:if value="${ros2_control_hardware_type == 'real'}">
+                    <plugin>topic_based_ros2_control/TopicBasedSystem</plugin>
+                    <param name="joint_commands_topic">/real_joint_commands</param>
+                    <param name="joint_states_topic">/real_joint_states</param>
+                </xacro:if>
             </hardware>
             <joint name="shoulder_pan">

File: config/so101_new_calib.urdf.xacro (robot description, xacro)
@@ -2,8 +2,9 @@
 <robot xmlns:xacro="http://www.ros.org/wiki/xacro" name="so101_new_calib">
     <xacro:arg name="initial_positions_file" default="initial_positions.yaml" />
+    <xacro:arg name="ros2_control_hardware_type" default="mock_components" />
     <!-- Import so101_new_calib urdf file -->
     <xacro:include filename="$(find so101_moveit2_description)/model/so101_arm.urdf" />
     <!-- Import control_xacro -->
     <xacro:include filename="so101_new_calib.ros2_control.xacro" />
-    <xacro:so101_new_calib_ros2_control name="FakeSystem" initial_positions_file="$(arg initial_positions_file)"/>
+    <xacro:so101_new_calib_ros2_control name="FakeSystem" initial_positions_file="$(arg initial_positions_file)" ros2_control_hardware_type="$(arg ros2_control_hardware_type)"/>
 </robot>
